Commit message: Replace mesh geometries with box geometries in URDF files for fr3v5, fr3v6, fr5v6, and fr10v6

File: frcobot_description/urdf/fr10v6.urdf (robot description, URDF)
Before this commit: robot fr10v6, 9 links, 8 joints
Links:
- link tool_Link: geometry collision box size=0 0 0; visual box size=0 0 0

File: frcobot_description/urdf/fr3v5.urdf (robot description, URDF)
Before this commit: robot fr3v5, 9 links, 8 joints
Links:
- link tool_Link: geometry collision box size=0 0 0; visual box size=0 0 0

File: frcobot_description/urdf/fr3v6.urdf (robot description, URDF)
Before this commit: robot fr3v6, 9 links, 8 joints
Links:
- link tool_Link: geometry collision box size=0 0 0; visual box size=0 0 0

File: frcobot_description/urdf/fr5v6.urdf (robot description, URDF)
Before this commit: robot fr5v6, 9 links, 8 joints
Links:
- link tool_Link: geometry collision box size=0 0 0; visual box size=0 0 0
